Commit message: Update model to new version

File: urdf/simple_mockup.urdf (robot description, URDF)
Before this commit: robot simple_mockup, 5 links, 4 joints
Joints:
- joint bar_hor: origin xyz=0.0 0.0 5.960464477539063e-08 rpy=1.5707963705062866 0.0 0.0 -> xyz=0.0 0.0 2.384185791015625e-07 rpy=1.5707963705062866 0.0 0.0
- joint bar_inc: origin xyz=0.0 -2.9802322387695312e-08 0.0 rpy=1.5707963705062866 -0.7853981852531433 0.0 -> xyz=0.0 -5.960464477539063e-08 0.0 rpy=1.5707963705062866 -0.7853981852531433 0.0
- joint bar_ver: origin xyz=5.960464477539063e-08 -2.9802322387695312e-08 0.0 rpy=1.5707963705062866 0.0 0.0 -> xyz=0.0 0.0 -1.0587911840678754e-22 rpy=1.5707963705062866 0.0 0.0

Commit message: Fix model orientation for registration

File: urdf/simple_mockup.urdf (robot description, URDF)
Before this commit: robot simple_mockup, 5 links, 4 joints
Joints:
- joint bar_hor: origin xyz=0.0 0.0 2.384185791015625e-07 rpy=1.5707963705062866 0.0 0.0 -> xyz=0.0 0.0 0.0 rpy=0.0 0.0 0.0
- joint bar_inc: origin xyz=0.0 -5.960464477539063e-08 0.0 rpy=1.5707963705062866 -0.7853981852531433 0.0 -> xyz=0.0 0.0 0.0 rpy=0.0 0.0 0.0
- joint bar_ver: origin xyz=0.0 0.0 -1.0587911840678754e-22 rpy=1.5707963705062866 0.0 0.0 -> xyz=0.0 0.0 0.0 rpy=0.0 0.0 0.0
- joint wall: origin xyz=0.0 0.0 0.0 rpy=1.5707963705062866 0.0 0.0 -> xyz=0.0 0.0 0.0 rpy=0.0 0.0 0.0

Commit message: Visual and collision shapes for the nappe manipulation

File: urdf/simple_mockup.urdf (robot description, URDF)
Before this commit: robot simple_mockup, 5 links, 4 joints
Links:
- added link LowerBox; collision box size=0.65 0.72 0.62; visual box size=0.65 0.72 0.62
- added link MiddleCylinder; collision cylinder length=0.62 radius=0.03; visual cylinder length=0.62 radius=0.03
- added link TopCylinder; collision cylinder length=0.62 radius=0.03; visual cylinder length=0.62 radius=0.03
Joints:
- added joint LowerBoxJoint: type fixed, parent base_link, child LowerBox, origin xyz=0.9 0.0 0.35 rpy=1.57 0.0 0.0
- added joint MiddleCylinderJoint: type fixed, parent base_link, child MiddleCylinder, origin xyz=1.08 0.0 1.12 rpy=1.57 0.0 0.0
- added joint TopCylinderJoint: type fixed, parent base_link, child TopCylinder, origin xyz=0.98 0.0 1.02 rpy=1.57 0.0 0.0

Commit message: Add horizontal cylinder

File: urdf/simple_mockup.urdf (robot description, URDF)
Before this commit: robot simple_mockup, 8 links, 7 joints
Links:
- added link CylinderBarTop; collision cylinder length=0.18 radius=0.02; visual cylinder length=0.18 radius=0.02
Joints:
- added joint CylinderBarTop: type fixed, parent base_link, child CylinderBarTop, origin xyz=1 0.30 1.12 rpy=0.0 1.57 0.0

Commit message: Rename to Cylinder*

File: urdf/simple_mockup.urdf (robot description, URDF)
Before this commit: robot simple_mockup, 9 links, 8 joints
Links:
- removed link MiddleCylinder
- removed link TopCylinder
- added link CylinderMiddle; collision cylinder length=0.62 radius=0.03; visual cylinder length=0.62 radius=0.03
- added link CylinderTop; collision cylinder length=0.62 radius=0.03; visual cylinder length=0.62 radius=0.03
Joints:
- removed joint MiddleCylinderJoint
- removed joint TopCylinderJoint
- added joint CylinderMiddleJoint: type fixed, parent base_link, child CylinderMiddle, origin xyz=1.08 0.0 1.12 rpy=1.57 0.0 0.0
- added joint CylinderTopJoint: type fixed, parent base_link, child CylinderTop, origin xyz=0.98 0.0 1.02 rpy=1.57 0.0 0.0
